Commit message: Add image processing to find location of robot and generate path.

File: src/robot_description/urdf/diff_wheeled_robot.xacro (robot description, xacro)
@@ -44,5 +44,5 @@
   <property name="base_z_origin_to_wheel_origin" value="0.0" />
   <!-- Hokuyo Laser scanner -->
-  <property name="hokuyo_size" value="0.05" />
+  <property name="hokuyo_size" value="0.07" />
   <!-- Macro for calculating inertia of cylinder -->
   <macro name="cylinder_inertia" params="m r h">
@@ -179,5 +179,5 @@
         <origin xyz="0 0 0" rpy="0 0 0" />
         <geometry>
-          <cylinder length="${hokuyo_size}" radius="${hokuyo_size/2}"/>
+          <cylinder length="${hokuyo_size/2}" radius="${hokuyo_size/2}"/>
         </geometry>
         <material name="Blue" />
@@ -185,5 +185,5 @@
     </link>
     <joint name="hokuyo_joint" type="fixed">
-      <origin xyz="${base_radius - hokuyo_size/2} 0 ${base_height+hokuyo_size/4}" rpy="0 0 0" />
+      <origin xyz="${base_radius - hokuyo_size} 0 ${base_height+hokuyo_size/8}" rpy="0 0 0" />
       <parent link="base_link"/>
       <child link="hokuyo_link" />
